Commit message: Big Push

File: src/forklift_simulator/urdf/RX20_16/base.xacro (robot description, xacro)
@@ -24,4 +24,5 @@
     </visual>
   </link>
+  <link name="imu_link"/>
   <joint name="imu_joint" type="fixed">
     <parent link="base_link"/>
@@ -29,5 +30,4 @@
     <origin xyz="0.0 0 0.068" rpy="0 0 0"/>
   </joint>
-  <link name="imu_link"/>
   <joint name="base_joint" type="fixed">
     <parent link="base_footprint" />
@@ -36,5 +36,5 @@
     <axis xyz="0 0 1" />
   </joint>
-  <joint name="scan_joint" type="fixed">
+  <joint name="scan" type="fixed">
     <parent link="base_footprint" />
     <child link="base_scan" />

File: src/forklift_simulator/urdf/RX20_16/d435_sensor.xacro (robot description, xacro)
@@ -36,4 +36,7 @@
           </clip>
           <noise>
+            <type>gaussian</type>
+            <mean>0.0</mean>
+            <stddev>0.007</stddev>
             <type>gaussian</type>
             <mean>0.0</mean>

File: src/forklift_simulator/urdf/RX20_16/front_wheels.xacro (robot description, xacro)
@@ -1,52 +1,52 @@
 <?xml version="1.0" ?>
-<robot name="RX20_16" xmlns:xacro="http://www.ros.org/wiki/xacro">
-<xacro:macro name="rx20_front_wheel" params="name x_loading y_loading z_loading radius width flip">
-  <link name="wheel_${name}_driving_link">
-    <inertial>
-    <origin xyz="0 0 0" rpy="0 0 0"/>
-    <xacro:cylinder_inertia mass="1" r="${radius}" l="${width}" />
-    <mass value= "1"/>
-    </inertial>
-    <collision >
+<robot name="RX20_16" xmlns:xacro="http://www.ros.org/wiki/xacro" >
+  <xacro:macro name="front_wheel" params="name parent x_loading y_loading z_loading radius width flip">
+    <link name="wheel_${name}_driving_link">
+      <inertial>
+      <origin xyz="0 0 0" rpy="0 0 0"/>
+      <xacro:cylinder_inertia mass="1" r="${radius}" l="${width}" />
+      <mass value= "1"/>
+      </inertial>
+      <collision >
+        <origin xyz="0 0 0" rpy="0 0 0"/>
+        <geometry>
+            <cylinder radius="${radius}" length="${width}"/>
+        </geometry>
+      </collision>
+      <visual>
       <origin xyz="0 0 0" rpy="0 0 0"/>
       <geometry>
-           <cylinder radius="${radius}" length="${width}"/>
+          <mesh filename="$(find forklift_simulator)/urdf/RX20_16/meshes/front_wheel.dae" />
       </geometry>
-    </collision>
-    <visual>
-    <origin xyz="0 0 0" rpy="0 0 0"/>
-    <geometry>
-        <mesh filename="$(find forklift_simulator)/urdf/RX20_16/meshes/front_wheel.dae" />
-    </geometry>
-    </visual>
-  </link>
-  <joint name="wheel_${name}_driving_joint" type="continuous">
-    <parent link="base_link" />
-    <child link="wheel_${name}_driving_link" />
-    <origin xyz="${x_loading} ${y_loading} ${z_loading}" rpy="1.57 0 0" />
-    <axis xyz="0 0 ${1*flip}" />
-    <!-- <joint_properties damping="1.0" friction="1.0"/> -->
-    <limit effort="100" velocity="100"/>
-     <dynamics damping="0.01" friction="1.0"/>
-  </joint>
-   <transmission name="trans_dynamic_${name}">
-    <type>transmission_interface/SimpleTransmission</type>
-    <joint name="wheel_${name}_driving_joint">
-      <hardwareInterface>hardware_interface/EffortJointInterface</hardwareInterface>
+      </visual>
+    </link>
+    <joint name="wheel_${name}_driving_joint" type="continuous">
+      <parent link="${parent}_link" />
+      <child link="wheel_${name}_driving_link" />
+      <origin xyz="${x_loading} ${y_loading} ${z_loading}" rpy="1.57 0 0" />
+      <axis xyz="0 0 ${1*flip}" />
+      <!-- <joint_properties damping="1.0" friction="1.0"/> -->
+      <limit effort="100" velocity="100"/>
+      <dynamics damping="0.01" friction="1.0"/>
     </joint>
-    <actuator name="motor_dynamic_wheel_${name}">
-      <hardwareInterface>hardware_interface/EffortJointInterface</hardwareInterface>
-      <mechanicalReduction>1</mechanicalReduction>
-    </actuator>
-  </transmission>
-  <gazebo reference="wheel_${name}_driving_link">
-			<mu1>1.0</mu1>
-			<mu2>1.0</mu2>
-			<!-- <kp>10000000.0</kp> -->
-			<kp>1000000000.0</kp>
-			<kd>1000.0</kd>
-			<minDepth>0.002</minDepth>
-			<maxVel>0</maxVel>
-		</gazebo>
- </xacro:macro>
+    <transmission name="trans_dynamic_${name}">
+      <type>transmission_interface/SimpleTransmission</type>
+      <joint name="wheel_${name}_driving_joint">
+        <hardwareInterface>hardware_interface/VelocityJointInterface</hardwareInterface>
+      </joint>
+      <actuator name="motor_dynamic_wheel_${name}">
+        <hardwareInterface>hardware_interface/VelocityJointInterface</hardwareInterface>
+        <mechanicalReduction>1</mechanicalReduction>
+      </actuator>
+    </transmission>
+    <gazebo reference="wheel_${name}_driving_link">
+        <mu1>1.0</mu1>
+        <mu2>1.0</mu2>
+        <!-- <kp>10000000.0</kp> -->
+        <kp>1000000000.0</kp>
+        <kd>1000.0</kd>
+        <minDepth>0.002</minDepth>
+        <maxVel>0</maxVel>
+      </gazebo>
+  </xacro:macro>
 </robot>

File: src/forklift_simulator/urdf/RX20_16/loading_forklift_joints.xacro (robot description, xacro)
@@ -169,3 +169,3 @@
     <axis xyz="0 0 1" />
   </joint>
-  </robot>
+</robot>

File: src/forklift_simulator/urdf/RX20_16/main.xacro (robot description, xacro)
@@ -1,22 +1,103 @@
 <?xml version="1.0" ?>
-<robot name="RX20_16" xmlns:xacro="http://www.ros.org/wiki/xacro" >
-<xacro:include filename="$(find forklift_simulator)/urdf/RX20_16/inertia.xacro" />
-<xacro:include filename="$(find forklift_simulator)/urdf/RX20_16/base.xacro" />
-<xacro:include filename="$(find forklift_simulator)/urdf/RX20_16/nav_lidar.xacro" />
-<xacro:include filename="$(find forklift_simulator)/urdf/RX20_16/detection_lidar.xacro" />
-<xacro:include filename="$(find forklift_simulator)/urdf/RX20_16/steer_wheels.xacro" />
-<xacro:include filename="$(find forklift_simulator)/urdf/RX20_16/front_wheels.xacro" />
-<xacro:include filename="$(find forklift_simulator)/urdf/RX20_16/d435_camera.xacro" />
-<xacro:include filename="$(find forklift_simulator)/urdf/RX20_16/loading_forklift_joints.xacro" />
-<xacro:include filename="$(find forklift_simulator)/urdf/RX20_16/lib_ackermansteer.xacro" />
-<xacro:camera_d435 name="camera" topics_ns="camera" parent="lift_link" publish_pointcloud="true"> <origin xyz="0.02 0 0.1" rpy="0 0 0" /> </xacro:camera_d435>
-<xacro:rx20_steer_wheel name="left" x_steering="-1.429" y_steering="0.404" z_steering="0.06" radius="0.150" width="0.15" flip="-1" />
-<xacro:rx20_steer_wheel name="right" x_steering="-1.429" y_steering="-0.404" z_steering="0.06" radius="0.150" width="0.15" flip="-1" />
-<xacro:rx20_front_wheel name="right" x_loading="0.0" y_loading="0.466" z_loading="0.0" radius="0.18" width="0.18" flip="-1" />
-<xacro:rx20_front_wheel name="left" x_loading="0.0" y_loading="-0.466" z_loading="0.0" radius="0.18" width="0.18" flip="-1" />
-<!-- <xacro:nav_lidar name="one"  x="0.5"  y="0.0" z="1.8" roll="0" pitch="0" yaw="0.0" resolution="1"/> -->
-<!-- <xacro:detection_lidar name="front"  x="0.0"  y="0.0" z="2.0" roll="0" pitch="0" yaw="0" resolution="1"/> -->
-<xacro:nav_lidar name="back"  x="0.2"  y="-0.6" z="-0.1" roll="0" pitch="0" yaw="1.57" resolution="1"/>
-<!-- <xacro:nav_lidar name="front"  x="0"  y="0.4" z="0.1" roll="0" pitch="0" yaw="-1.57" resolution="1"/> -->
-<!-- <xacro:detection_lidar name="front"  x="0.0"  y="0.0" z="0.6" roll="0" pitch="0" yaw="0" resolution="1"/> -->
+<robot name="RX20_16" xmlns:xacro="http://www.ros.org/wiki/xacro">
+  <xacro:property name="deg_to_rad" value="0.01745329251994329577"/>
+  <!-- Robot base dimensions -->
+  <xacro:property name="base_length" value="-1.839" /> <!--fake 0.5 real 0.139-->
+  <xacro:property name="base_width" value="1.1" /> <!--fake 0.3 real 0.139-->
+  <xacro:property name="base_height" value="0.835" /> <!--fake 0.1 real 0.139-->
+  <xacro:property name="base_mass" value="10" />
+  <!-- Wheel link dimensions -->
+  <xacro:property name="wheel_radius" value="0.10" /> <!--fake 0.1 real 0.139-->
+  <xacro:property name="wheel_thickness" value=".13" /> <!--fake 0.08 real 0.139-->
+  <xacro:property name="wheel_mass" value="1" />
+  <!-- Steering link dimensions -->
+  <xacro:property name="steer_radius" value="0.05" />
+  <xacro:property name="steer_height" value="0.12" />
+  <xacro:property name="steer_thickness" value="0.02" />
+  <xacro:property name="steer_mass" value="1" />
+  <!-- Axle positions -->
+  <xacro:property name="axle_offset" value="0.036175" /> <!--fake 0.05 real 0.035-->
+  <xacro:property name="steer_offset" value="0.0254" /> <!--fake 0.02 real 0.139-->
+  <!--<gazebo>
+    <plugin name="gazebo_ros_control" filename="libgazebo_ros_control.so">
+      <robotNamespace>"/RX20_16"</robotNamespace>
+      <robotSimType>steer_bot_hardware_gazebo/SteerBotHardwareGazebo</robotSimType>
+      <legacyModeNS>false</legacyModeNS>
+    </plugin>
+  </gazebo>-->
+    <xacro:include filename="$(find forklift_simulator)/urdf/RX20_16/inertia.xacro" />
+    <xacro:include filename="$(find forklift_simulator)/urdf/RX20_16/base.xacro" />
+    <xacro:include filename="$(find forklift_simulator)/urdf/RX20_16/nav_lidar.xacro" />
+    <xacro:include filename="$(find forklift_simulator)/urdf/RX20_16/detection_lidar.xacro" />
+    <xacro:include filename="$(find forklift_simulator)/urdf/RX20_16/d435_camera.xacro" />
+    <xacro:include filename="$(find forklift_simulator)/urdf/RX20_16/inertials.xacro" />
+    <xacro:include filename="$(find forklift_simulator)/urdf/RX20_16/loading_forklift_joints.xacro" />
+    <xacro:include filename="$(find forklift_simulator)/urdf/RX20_16/rear_steer.xacro" />
+    <xacro:include filename="$(find forklift_simulator)/urdf/RX20_16/steer_wheels.xacro" />
+    <xacro:camera_d435 name="camera" topics_ns="camera" parent="lift_link" publish_pointcloud="true"> <origin xyz="0.02 0 0.1" rpy="0 0 0" /> </xacro:camera_d435>
+    <!--<xacro:detection_lidar name="front"  x="0.0"  y="0.0" z="2.0" roll="0" pitch="0" yaw="0" resolution="1"/>-->
+    <xacro:nav_lidar name="back"  x="0.4"  y="0.0" z="-0.08" roll="0.0" pitch="0.0" yaw="0" resolution="1"/>
+    <!--<xacro:nav_lidar name="front"  x="0"  y="0.4" z="0.1" roll="0" pitch="0" yaw="-1.57" resolution="1"/-->
+    <!-- <xacro:detection_lidar name="front"  x="0.0"  y="0.0" z="0.6" roll="0" pitch="0" yaw="0" resolution="1"/> -->
+ <xacro:rear_steer
+    name="rear"
+    parent="base"
+    steer_radius="${steer_radius}"
+    steer_thickness="${steer_thickness}"
+    steer_mass="${steer_mass}"
+    base_length="${base_length}"
+    base_width="${base_width}"
+    axle_offset="${axle_offset}"
+    steer_height="${steer_height-.06}">
+</xacro:rear_steer>
+ <xacro:rear_wheel
+    name="front"
+    parent="base"
+    wheel_radius="${wheel_radius/4}"
+    wheel_thickness="${base_width}"
+    wheel_mass="${wheel_mass}">
+    <origin xyz="0 0 0" rpy="${-90 * deg_to_rad} 0 0"/>
+  </xacro:rear_wheel>
+   <xacro:steer_wheel name="rear_left"  x_steering="-1.429" y_steering="0.404" z_steering="0.06" radius="0.150" width="0.15" flip="-1" />
+   <xacro:steer_wheel name="rear_right" x_steering="-1.429" y_steering="-0.404" z_steering="0.06" radius="0.150" width="0.15" flip="-1" />
+   <!-- <xacro:rear_wheel_lr
+    name="rear_right"
+    parent="base"
+    reflect="-1"
+    x_steering="-1.429"
+    y_steering="-0.404"
+    z_steering="0.06"
+    wheel_radius="${wheel_radius}"
+    wheel_thickness="${wheel_thickness}"
+    wheel_mass="${wheel_mass}"
+    steer_radius="${steer_radius}"
+    steer_thickness="${steer_thickness}"
+    steer_mass="${steer_mass}"
+    base_length="${base_length}"
+    base_width="${base_width}"
+    axle_offset="${axle_offset}"
+    steer_height="${steer_height}"
+    flip = "-1">
+  </xacro:rear_wheel_lr>
+  <xacro:rear_wheel_lr
+    name="rear_left"
+    parent="base"
+    reflect="1"
+    x_steering="-1.429"
+    y_steering="0.404"
+    z_steering="0.06"
+    wheel_radius="${wheel_radius}"
+    wheel_thickness="${wheel_thickness}"
+    wheel_mass="${wheel_mass}"
+    steer_radius="${steer_radius}"
+    steer_thickness="${steer_thickness}"
+    steer_mass="${steer_mass}"
+    base_length="${base_length}"
+    base_width="${base_width}"
+    axle_offset="${axle_offset}"
+    steer_height="${steer_height}"
+    flip = "-1">
+  </xacro:rear_wheel_lr>-->
+    <xacro:front_wheel_lr name="front_right" parent = "base" x_loading="0.0" y_loading="-0.466" z_loading="0.0" radius="0.18" width="0.18" flip="-1" />
+    <xacro:front_wheel_lr name="front_left" parent = "base" x_loading="0.0" y_loading="0.466" z_loading="0.0" radius="0.18" width="0.18" flip="-1" />
 </robot>

File: src/forklift_simulator/urdf/RX20_16/nav_lidar.xacro (robot description, xacro)
@@ -54,7 +54,8 @@
         <plugin filename="libgazebo_ros_laser.so"   name="gazebo_ros_head_hokuyo_controller">
           <!-- <topicName>/${name}_nav_lidar</topicName> -->
-          <topicName>/scan</topicName>
+          <topicName>/RX20_16/scan</topicName>
             <frameName>${name}_nav_lidar</frameName>
-            <!-- <frameName>base_footprint</frameName> -->
+            <!-- <frameName>base_footprint</frameName> -->_
+          <output_type>sensor_msgs/LaserScan</output_type>
         </plugin>
       </sensor>

File: src/forklift_simulator/urdf/RX20_16/steer_wheels.xacro (robot description, xacro)
@@ -1,6 +1,6 @@
 <?xml version="1.0" ?>
 <robot name="RX20_16" xmlns:xacro="http://www.ros.org/wiki/xacro">
-<xacro:macro name="rx20_steer_wheel" params="name x_steering y_steering z_steering radius width flip">
-  <link name="wheel_${name}_steering_link">
+<xacro:macro name="steer_wheel" params="name x_steering y_steering z_steering radius width flip">
+  <link name="${name}_steer_link">
     <inertial>
     <origin xyz="0 0 0.1125" rpy="0 0 0"/>
@@ -21,7 +21,7 @@
     </visual>
   </link>
-  <joint name="wheel_${name}_steering_joint" type="revolute">
-    <parent link="base_link" />
-    <child link="wheel_${name}_steering_link" />
+    <joint name="${name}_steer_joint" type="revolute">
+      <parent link="base_link"/>
+      <child link="${name}_steer_link"/>
     <origin xyz="${x_steering} ${y_steering} ${z_steering }" rpy="0 0 1.57" />
     <!-- <origin xyz="-0.662 0.247 0.115" rpy="0 0 0" /> -->
@@ -30,5 +30,5 @@
      <dynamics damping="1" friction="1"/>
   </joint>
-  <link name="wheel_${name}_link">
+  <link name="${name}_wheel_link">
     <inertial>
     <origin xyz="0 0 0" rpy="0 0 0"/>
@@ -50,19 +50,19 @@
     </visual>
   </link>
-  <joint name="wheel_${name}_joint" type="continuous">
-    <parent link="wheel_${name}_steering_link" />
-    <child link="wheel_${name}_link" />
-    <origin xyz=" 0 0 -0.09" rpy="0 1.57 0" />
-    <axis xyz="0 0 1" />
+  <joint name="${name}_wheel_joint" type="continuous">
+      <parent link="${name}_steer_link"/>
+      <child link="${name}_wheel_link"/>
+    <origin xyz=" 0 0 -0.09" rpy="0 1.57 0"/>
+    <axis xyz="0 0 1"/>
     <!-- <joint_properties damping="1.0" friction="0.3"/> -->
-        <limit effort="100" velocity="100"/>
-     <dynamics damping="0.01" friction="0.0"/>
+        <limit effort="10" velocity="10"/>
+     <dynamics damping="0.01" friction="0.3"/>
   </joint>
   <transmission name="trans_steering_${name}">
     <type>transmission_interface/SimpleTransmission</type>
-    <joint name="wheel_${name}_steering_joint">
+    <joint name="${name}_steer_joint">
       <hardwareInterface>hardware_interface/EffortJointInterface</hardwareInterface>
     </joint>
-    <actuator name="motor_steering_wheel_${name}">
+    <actuator name="${name}_steer_joint_motor">
       <hardwareInterface>hardware_interface/EffortJointInterface</hardwareInterface>
       <mechanicalReduction>1</mechanicalReduction>
